File: KiCAD Design/KiCAD Design.kicad_pcb (KiCad board)
At the start: 2 copper layers, 51 x 60.5 mm, 60 parts, among them J1 USB_B_Micro, J2 Conn_01x04_Pin, J5 Micro_SD_Card, SW1 SW_SPDT, U1 STM32F103C8Tx, U2 AMS1117-3.3, U3 BNO055, U4 L80-R, U5 nRF24L01P, Y1 16MHz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

Commit message: All layout finished, ready to prep for order
Parts:
- moved H1 6.67 mm to (146.2, 71.5)
- moved H3 6.58 mm to (146.2, 123.5)
- moved C12 3.90 mm to (174.0, 88.5)
- moved H2 2.92 mm to (182.2, 71.5)
- moved H4 2.69 mm to (182.2, 123.5)
- moved J1 2.41 mm to (181.3, 95.0)
- moved R7 2.13 mm to (156.8, 107.0)
- moved R9 1.50 mm to (159.8, 107.0)
- moved R10 1.42 mm to (160.8, 108.2), turned to 0 degrees
- moved J2 1.24 mm to (177.6, 72.0)
- moved R8 1.13 mm to (155.8, 108.2), turned to 180 degrees
Connections:
- J1 pad 6: unconnected-(J1-Shield-Pad6) -> (no net)
- U5 pad 21: GND -> (no net)
Routing:
- net +3.3V: track 64.2 -> 205.3 mm, vias 0 -> 19
- net Antenna: track 0.00 -> 37.1 mm
- net SPI1_SCK: track 4.76 -> 25.8 mm
- net SD_CD: track 3.94 -> 19.0 mm
- net SPI1_MISO: track 9.15 -> 20.9 mm
- net SPI1_MOSI: track 8.72 -> 18.8 mm
- net GND: track 107.6 -> 100.6 mm, vias 33 -> 36
- net SPI2_SCK: track 5.47 -> 8.65 mm, vias 0 -> 2
- net UART3_TX: track 19.3 -> 22.1 mm
- net VBUS: track 3.04 -> 5.82 mm, vias 0 -> 2
- net /USB_D+: track 14.3 -> 16.7 mm
- net /USB_D-: track 14.3 -> 16.7 mm
- net /SWDIO: track 32.8 -> 31.5 mm
- net /SWCLK: track 28.6 -> 27.3 mm
- net SPI2_IRQ: track 6.87 -> 5.88 mm
- added copper zone on F.Cu, net +3.3V
- added copper zone on F.Cu, net GND
- added copper zone on F.Cu, net VBUS
Other:
- board size 51 x 60.5 mm -> 42 x 58 mm

Commit message: Assembly files
Parts:
- removed C14, C15, C16: 100n, Capacitor_SMD:C_0402_1005Metric
- removed U3: BNO055, Package_LGA:LGA-28_5.2x3.8mm_P0.5mm
- added J3: Conn_01x04_Pin, Connector_PinHeader_2.54mm:PinHeader_1x04_P2.54mm_Vertical, F.Cu at (146.2, 107.0)
Connections:
- J1 pad 6: (no net) -> unconnected-(J1-Shield-Pad6)
- U1 pad 12: UART2_TX -> /UART2_TX
- U1 pad 13: UART2_RX -> /UART2_RX
Routing:
- net UART2_RX: track 24.9 -> 0.00 mm
- net /UART2_RX: track 0.00 -> 14.7 mm
- net /UART2_TX: track 0.00 -> 13.1 mm
- net IMU_INT: track 10.1 -> 0.00 mm
- net UART2_TX: track 10.1 -> 0.00 mm
- net +3.3V: track 205.3 -> 197.2 mm, vias 19 -> 18
- net GND: track 100.6 -> 93.2 mm, vias 36 -> 32
- net Net-(U3-CAP): track 1.34 -> 0.00 mm
Other:
- board text added: "UART"
